File: KiCAD/RC-MultiSwitcher.kicad_pcb (KiCad board)
At the start: 2 copper layers, 33 x 45.1 mm, 28 parts, among them IC1 LM2940IMP-5.0_NOPB, J1 Pwr_Outputs, J3 Srv_INPUTS, J4 Srv_OUTPUTS, Q1 DMG9926USD-13, Q2 DMG9926USD-13, Q3 DMG9926USD-13, U1 Teensy3.1

Commit message: minor layout improvements; added manufacturing data
Parts:
- C1: value 0.47µF/16V -> 470nF/50V
- U1: value Teensy3.1 -> Teensy3.1_Minimal
- moved R4 5.85 mm to (138.4, 87.6), turned to 90 degrees
- moved R3 4.44 mm to (142.2, 92.7), turned to 90 degrees
- moved R9 2.54 mm to (142.2, 80.6), turned to 90 degrees
- moved R1 1.42 mm to (137.2, 98.4)
- moved F1 0.64 mm to (135.9, 92.1)
- moved R2 0.63 mm to (137.2, 96.5)
Routing:
- net Net-(Q2-Pad4): track 6.68 -> 12.5 mm, vias 0 -> 1
- net GND: track 29.6 -> 27.5 mm
- net Net-(Q1-Pad2): track 34.4 -> 32.8 mm
- net Net-(Q2-Pad2): track 17.5 -> 18.7 mm
- net /SW3: track 25.1 -> 24.0 mm
- net +5V: track 17.9 -> 17.1 mm
- net Net-(Q1-Pad4): track 29.7 -> 29.0 mm
- net /PWR-IN: track 11.8 -> 12.5 mm
- net /SW6: vias 2 -> 1
Other:
- board text added: "RC-MultiSwitcher v1.0"
- board text added: "github.com/juepi"

Commit message: minor update to PCB
Parts:
- added J2: Alt_Pwr, Connector_JST:JST_XH_B2B-XH-A_1x02_P2.50mm_Vertical, F.Cu at (134.1, 92.7)
- added JP2: , Jumper:SolderJumper-2_P1.3mm_Open_Pad1.0x1.5mm, B.Cu at (135.3, 98.4)
- moved F1 6.38 mm to (135.3, 98.4), turned to 0 degrees
- moved R2 6.35 mm to (137.2, 102.9)
- moved R1 5.72 mm to (137.2, 104.1)
- moved R11 1.91 mm to (138.4, 82.5)
- moved R4 1.91 mm to (138.4, 85.7)
Routing:
- net /PWR-IN: track 12.5 -> 24.1 mm
- net Net-(Q1-Pad4): track 29.0 -> 35.3 mm
- net Net-(Q1-Pad2): track 32.8 -> 38.6 mm
- net Net-(Q2-Pad4): track 12.5 -> 13.2 mm
- net /I-SRV0: track 7.10 -> 6.58 mm
Other:
- board text added: "RC-MultiSwitcher v1.1"
- board text removed: "RC-MultiSwitcher v1.0"

Commit message: major code updates
Connections:
- D1 pad 2: /SW1 -> /SW0
- D2 pad 2: /SW2 -> /SW1
- D3 pad 2: /SW3 -> /SW2
- D4 pad 2: /SW4 -> /SW3
- D5 pad 2: /SW5 -> /SW4
- D6 pad 2: /SW6 -> /SW5
- J1 pad 1: /SW1 -> /SW0
- J1 pad 11: /SW6 -> /SW5
- J1 pad 3: /SW2 -> /SW1
- J1 pad 5: /SW3 -> /SW2
- J1 pad 7: /SW4 -> /SW3
- J1 pad 9: /SW5 -> /SW4
- Q1 pad 5: /SW2 -> /SW1
- Q1 pad 6: /SW2 -> /SW1
- Q1 pad 7: /SW1 -> /SW0
- Q1 pad 8: /SW1 -> /SW0
- Q2 pad 5: /SW4 -> /SW3
- Q2 pad 6: /SW4 -> /SW3
- Q2 pad 7: /SW3 -> /SW2
- Q2 pad 8: /SW3 -> /SW2
- Q3 pad 5: /SW6 -> /SW5
- Q3 pad 6: /SW6 -> /SW5
- Q3 pad 7: /SW5 -> /SW4
- Q3 pad 8: /SW5 -> /SW4
Routing:
- net /SW6: track 30.0 -> 0.00 mm, vias 1 -> 0
- net /SW0: track 0.00 -> 24.6 mm
- net /SW1: track 24.6 -> 20.8 mm, vias 0 -> 1
- net /SW5: track 26.1 -> 30.0 mm, vias 0 -> 1
- net /SW4: track 22.4 -> 26.1 mm, vias 1 -> 0
- net /SW2: track 20.8 -> 24.0 mm, vias 1 -> 0
- net /SW3: track 24.0 -> 22.4 mm, vias 0 -> 1
